File: fadecandybreakout.sch (EAGLE design)
At the start: 16 parts

Commit message: Initial Commit
Other:
- note added: "Catalyze Chicago"
- note added: "R1"
- moved on the sheet: FAT_GND, FAT_VCC, H1, H2, H3, H4, JP1, JP2, U$1, U$2, U$3, U$4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
